File: ATS-20/ATS-20_TB5CVN_Trace/ATS-20_TB5CVN_Trace.kicad_sch (KiCad schematic)
At the start: 74 parts, among them J1 Conn_01x01_Male, J10 Conn_01x04_Male, J2 Conn_01x01_Male, J3 Conn_01x01_Male, J4 Conn_01x02_Male, J5 Conn_Coaxial, J6 AudioJack3_SwitchTR, J7 Conn_01x02_Male, J8 Conn_01x14, J9 Conn_01x04_Male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

Commit message: Some schematic corrections
Changed incorrectly identified components in audio section - inductors (ferrite beads maybe?) is now shown instead of capacitors
Parts:
- removed C18, C19, C20: C, symbol Device:C
- removed J4, J7: Conn_01x02_Male, symbol Connector:Conn_01x02_Male
- added J4, J7: Conn_01x02, symbol Connector_Generic:Conn_01x02
- added L2, L3, L4: L, symbol Device:L
- renumbered C21 to C18, C22 to C19, C23 to C20
Connections:
- net 3.3V_Digital: now also A1.17 (3V3)
- net FM_Earphone_Antenna: now also L4.1
- net GND: now also J4.2 (Pin_2), L4.2
- net at C17.2, R12.1: now also L3.1
- net at J6.R: now also L3.2
- net at J6.T: now also L2.2
- net at R14.2, U7.5 (Vo1): now also J7.2 (Pin_2)
- net at C2.2, SW1.2 (B), U1.5 (BAT): now also J4.1 (Pin_1)
- net at C16.2, R11.1: now also L2.1
- net at U7.8 (Vo2): now also J7.1 (Pin_1)
- no-connect marks 10 -> 22
